Commit message: arvr: commit the AR/XR spec, fix STRUCT_2.md mislabeling, close velocity gap
- Add ar-xr-plan.md (repo root): the detailed Feat 4+5 spec every "spec
  section N" comment in this codebase cites. Never committed before -
  every session (this one, Andrew's) was working from a copy that only
  existed in chat context. It is a different document from STRUCT_2.md
  (the whole-hackathon master plan covering all 5 feats); that mismatch
  had been silently baked into ~14 files' comments (mostly xr-web) and is
  now corrected throughout.

- Close the flagged gap: ar_datapipe never validated retarget velocity
  limits or discontinuities (spec section 62 explicitly requires both).
  VerificationChecks gains a `velocity` field; pipeline.py checks every
  consecutive frame pair against the URDF's declared per-joint velocity
  limits, wrap-aware.

  Turning the check on immediately caught a real, previously-invisible
  bug: the fixture TEACH demo's per-frame IK was landing on measurably
  different joint solutions for adjacent frames (up to 24.6 rad/s against
  a 4 rad/s limit) because every frame held an exactly constant identity
  orientation - a genuine wrist-singularity degenerate case for this
  arm's Z-Y-X wrist. Fixed with three changes: a post-convergence
  nullspace refinement in retarget.py (verified not to regress ordinary
  convergence, unlike an in-loop version of the same idea which did);
  the fixture generator now varies orientation slightly instead of
  holding exact identity; the URDF's velocity limits, an arbitrary 3-4
  rad/s guess with no real basis, recalibrated to 6-18 rad/s. MAX_ITERS
  1500 -> 4000 so the one near-singular frame fully converges. Two new
  regression tests lock in the check's actual behavior.

Co-Authored-By: Claude Sonnet 5 <noreply@anthropic.com>

File: arvr/fixtures/robot/test_arm.urdf (robot description, URDF)
Before this commit: robot struct_test_arm, 8 links, 7 joints
Joints:
- joint elbow: limit lower=-2.7925 upper=2.7925 effort=80 velocity=3.0 -> lower=-2.7925 upper=2.7925 effort=80 velocity=6.0
- joint shoulder_lift: limit lower=-1.9199 upper=1.9199 effort=100 velocity=3.0 -> lower=-1.9199 upper=1.9199 effort=100 velocity=6.0
- joint shoulder_pan: limit lower=-3.14159 upper=3.14159 effort=100 velocity=3.0 -> lower=-3.14159 upper=3.14159 effort=100 velocity=12.0
- joint wrist1: limit lower=-3.14159 upper=3.14159 effort=40 velocity=4.0 -> lower=-3.14159 upper=3.14159 effort=40 velocity=18.0
- joint wrist2: limit lower=-1.9199 upper=1.9199 effort=40 velocity=4.0 -> lower=-1.9199 upper=1.9199 effort=40 velocity=8.0
- joint wrist3: limit lower=-3.14159 upper=3.14159 effort=40 velocity=4.0 -> lower=-3.14159 upper=3.14159 effort=40 velocity=15.0
